File: hardware/20x20/pico_flight_20x20.kicad_pcb (KiCad board)
At the start: 2 copper layers, 28 x 28 mm, 45 parts, among them J1 USB_B_Micro, J2 Conn_01x02, J3 DEBUG, J4 ESC_AIKON32, J5 UART1, J6 UART2, J7 CAM, J8 VTX, U1 MCP1711T-33I_OT, U2 W25Q128JVS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

Commit message: latest board
Parts:
- removed the J5 at (-17.1, -11.1)
- added J5: UART1, pico-flight:PAD_X4_SMD_03x02, F.Cu at (22.6, 9.95)
- added J5: UART1, pico-flight:PAD_X4_SMD_03x02, F.Cu at (18.6, -2.67)
- added J5: UART1, pico-flight:PAD_X4_SMD_03x02, F.Cu at (11.0, -2.67)
- added J5: UART1, pico-flight:PAD_X4_SMD_03x02, F.Cu at (-2.48, 12.1)
- added J5: UART1, pico-flight:PAD_X4_SMD_03x02, F.Cu at (-2.48, 18.6)
- C18, C19, C20, U2: moved to B.Cu
- R1, R2: moved to F.Cu
- moved C5 15.1 mm to (21.8, 11.1), turned to 0 degrees
- moved U1 15.1 mm to (4.06, 6.60), turned to 180 degrees
- moved R1 8.55 mm to (19.7, 6.72), turned to 0 degrees
- moved U2 7.91 mm to (19.1, 6.46), turned to 0 degrees
- moved C3 7.22 mm to (1.52, 6.12), turned to 90 degrees
- moved C18 6.78 mm to (14.1, 1.93)
- moved C19 5.84 mm to (9.40, 3.30), turned to 270 degrees
- moved U4 5.54 mm to (12.0, 3.52)
- moved C20 5.30 mm to (9.96, 1.94)
- moved Y1 4.64 mm to (3.75, 6.74), turned to 90 degrees
- moved R2 3.97 mm to (16.6, 6.20), turned to 0 degrees
- moved C2 3.86 mm to (3.90, 10.8)
- moved R5 1.80 mm to (3.89, 11.8)
- moved R3 1.58 mm to (16.6, 12.8), turned to 180 degrees
- moved C1 1.07 mm to (22.0, 13.4)
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Routing:
- net +5V: track 0.00 -> 23.5 mm
- net +3V3: track 58.9 -> 38.4 mm, vias 8 -> 7
- net IMU_DATA_RDY: track 13.0 -> 2.10 mm, vias 2 -> 0
- net /QSPI_SD1: track 14.8 -> 5.30 mm, vias 2 -> 1
- net /QSPI_SD2: track 16.6 -> 7.92 mm, vias 0 -> 1
- net UART1_RX: track 0.93 -> 7.91 mm
- net Net-(C3-Pad1): track 3.12 -> 8.97 mm
- net IMU_SPI_CS: track 9.26 -> 3.59 mm, vias 2 -> 0
- net /QSPI_SD3: track 16.3 -> 10.8 mm, vias 2 -> 1
- net /QSPI_SD0: track 16.6 -> 11.4 mm, vias 2 -> 1
- net Net-(U3-Pad30): track 0.93 -> 5.38 mm
- net /QSPI_SS: track 13.2 -> 8.82 mm
- net /QSPI_SCLK: track 15.1 -> 11.0 mm, vias 2 -> 1
- net IMU_SPI_SCLK: track 8.13 -> 4.47 mm
- net Net-(U3-Pad29): track 0.96 -> 4.44 mm
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- removed copper zone on B.Cu, net +5V
