File: hardware/20x20/pico_flight_20x20.kicad_sch (KiCad schematic)
At the start: 54 parts, among them J1 USB_B_Micro, J2 Conn_01x02, J3 DEBUG, J4 ESC_AIKON32, J5 UART1, J6 UART2, J7 UART3, J8 UART4, U1 MCP1711T-33I_OT, U2 W25Q128JVS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

Commit message: latest kicad files
Parts:
- added C25: 10u, Capacitor_SMD:C_0603_1608Metric, symbol Device:C
- added D3: 5V_LED, LED_SMD:LED_0603_1608Metric, symbol Device:LED_Small
- added D4: 3V3_LED, LED_SMD:LED_0603_1608Metric, symbol Device:LED_Small
- added D5: STATUS, LED_SMD:LED_0603_1608Metric, symbol Device:LED_Small
- added R7, R8, R9: 2K, Resistor_SMD:R_0402_1005Metric, symbol Device:R_Small
- added U7: MCP1711T-33I_OT, Package_TO_SOT_SMD:SOT-23-5, symbol pico_flight_20x20-rescue:MCP1711T-33I_OT-2021-07-16_06-26-35
- C5: footprint Capacitor_SMD:C_0603_1608Metric -> Capacitor_SMD:C_0402_1005Metric
- J2: footprint Connector_PinHeader_2.54mm:PinHeader_1x02_P2.54mm_Vertical -> 01-pico-footprints:PAD_X2_SMD_01x02
- J5, J6, J7, J8: footprint pico-flight:PAD_X4_SMD_03x02 -> 01-pico-footprints:PAD_X4_SMD_03x02
- R1, R2, R6: footprint Resistor_SMD:R_0603_1608Metric -> Resistor_SMD:R_0402_1005Metric
- U1: footprint SOT-23-5_OT_MCH -> Package_TO_SOT_SMD:SOT-23-5
Connections:
- net +3V3: now also D4.1 (K); no longer C21.1, U5.13 (VDD)
- net +5V: now also D3.1 (K), U7.1 (VIN), U7.3 (*SHDN)
- net GND: now also C25.2, R7.2, R8.2, R9.2, U7.2 (GND)
- net IMU_DATA_RDY: now also U3.8 (GPIO6); no longer U3.6 (GPIO4)
- net UART1_RX: now also U3.7 (GPIO5); no longer U3.31 (GPIO20)
- net UART1_TX: now also U3.6 (GPIO4); no longer U3.32 (GPIO21)
- net RF_DIO_3: now reaches U3.11 (GPIO8)
- net RF_DIO_3: now also U4.10 (DIO3)
- net RF_DIO_2: now reaches U3.12 (GPIO9)
- net RF_DIO_2: now also U4.9 (DIO2)
- net RF_DIO_1: now reaches U3.13 (GPIO10)
- net RF_DIO_1: now also U4.8 (DIO1)
- net RF_BUSY: now reaches U3.14 (GPIO11)
- net RF_BUSY: now also U4.7 (BUSY)
- net RF_SPI_MISO: now reaches U3.15 (GPIO12)
- net RF_SPI_MISO: now also U4.16 (MISO_TX)
- net RF_SPI_CS: now reaches U3.16 (GPIO13)
- net RF_SPI_CS: now also U4.19 (NSS_CTS)
- net RF_SPI_SCLK: now reaches U3.17 (GPIO14)
- net RF_SPI_SCLK: now also U4.18 (SCK_RTSN)
- net RF_SPI_MOSI: now reaches U3.18 (GPIO15)
- net RF_SPI_MOSI: now also U4.17 (MOSI_RX)
- net RF_NRESET: now reaches U3.9 (GPIO7)
- net RF_NRESET: now also U4.3 (NRESET)
- new net: D5.1 (K), U3.32 (GPIO21)
- new net: D5.2 (A), R9.1
- new net: D3.2 (A), R7.1
- new net: D4.2 (A), R8.1
- new net +3.3VADC: C21.1, C25.1, U5.13 (VDD), U7.5 (VOUT)
- no-connect marks 5 -> 7
Other:
- moved on the sheet: C1, C10, C11, C12, C13, C14, C15, C16, C17, C2, C21, C3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
